Commit message: Gazebo world created

File: src/robot_description/urdf/arm.xacro (robot description, xacro)
@@ -12,5 +12,5 @@
     <collision>
       <geometry>
-        <mesh filename="package://robot_description/meshes/collision/link0.obj"/>
+        <mesh filename="package://robot_description/meshes/visual/link0.dae"/>
       </geometry>
     </collision>
@@ -36,5 +36,5 @@
     <collision>
       <geometry>
-        <mesh filename="package://robot_description/meshes/collision/link1.obj"/>
+        <mesh filename="package://robot_description/meshes/visual/link1.dae"/>
       </geometry>
     </collision>

Commit message: pymovit2 pkg created

File: src/robot_description/urdf/arm.xacro (robot description, xacro)
@@ -293,5 +293,5 @@
     <axis xyz="0 -1 0"/>
     <limit effort="30.0" lower="0.0" upper="0.04" velocity="10.0"/>
-    <!-- <mimic joint="panda_finger_joint1" multiplier="-1"/> -->
+    <!-- <mimic joint="panda_finger_joint1" multiplier="1" offset="0.0"/> -->
   </joint>
 </robot>
